File: cc2530-LR-standalone-router.sch (EAGLE design)
At the start: 12 parts, among them J1 629105150921, U1 AP2112K

Commit message: Modified Version (USB Stick)
Parts:
- removed J1: 629105150921, WR-USB_Rev20b:629105150921
- removed U1: AP2112K, SparkFun-IC-Power:V_REG_AP2112K-3.3V
- added L1: 33n, inductor-neosid:SM-1206
- added U2: MCP1703-3302, dersimn_basics:V_REG_SOT-22-3
- added X1: A-USB A-LP-SMT-C, dersimn_connector:USB-1.0/1.1/2.0-STANDARD-A/B_A-LP-SMT-C
- C1: value 1µ -> 4.7n; device rcl:C-EUC0805 -> rcl:C-EUC1206
- C2: value 1µ -> 10n; device rcl:C-EUC0805 -> rcl:C-EUC1206
- C3: value 100nF -> 1µF; device rcl:C-EUC0805 -> resistor:C-EUC1206
- C4: value 22u -> 1µF; device rcl:CPOL-EUC -> resistor:C-EUC1206
- R1: value 10k -> 1M; device rcl:R-EU_R0805 -> rcl:R-EU_R1206
- R2: device rcl:R-EU_R0805 -> rcl:R-EU_R1206
- STATUS: device led:LEDCHIPLED_0805 -> led:LEDCHIPLED_1206
- U$5: value E18-MS1PA1IPX -> E18-MS1PA2-PCB; device codm:E18-MS1PA1IPX -> e18-ms1pa1-ipx:E18-MS1PA2-PCB
Connections:
- removed net N$1: R1.2, U1.EN
- removed net VCC: C2.2, C3.2, DBGVCC.1, DEBUG.2, U$5.VCC, U1.OUT
- new net +3V3: C4.1, DBGVCC.1, DEBUG.2, U$5.VCC, U2.OUT
- new net SHIELD: C1.1, R1.1, X1.SHIELD
- new net VUSB: C2.1, L1.1, X1.VBUS
- net +5V: now also C3.1, L1.2, U2.IN; no longer C1.2, C4.+, J1.VBUS, R1.1, U1.IN
- net GND: now also C1.2, C2.2, C3.2, C4.2, R1.2, U2.GND, X1.GND; no longer C1.1, C2.1, C3.1, C4.-, J1.GND, J1.SHIELD, U1.GND
Other:
- note removed: "FK 22/16 AR"
- moved on the sheet: C1, C2, C3, DBGVCC, R1, R2, STATUS
